File: TrialBBConversion/TrialBBConversion.sch (KiCad schematic (older format))
At the start: 41 parts, among them SW1 SW_SPDT, SW2 SW_Push, SW3 SW_Push, U1 DRV883-MPV_Symbol_Lib, U2 Color_Sensor-MPV_Symbol_Lib, U3 a-24543.5mmAudio, U4 SPX3819M5-L-3-3, X1 Arduino_Pro_Mini

Commit message: new stuff
Parts:
- X1: symbol Arduino_Pro_Mini:Arduino_Pro_Mini -> TrialBBConversion-rescue:Arduino_Pro_Mini-Arduino_Pro_Mini
Changed lines of the file:
@@
 Connection ~ 4150 3550
 $Comp
-L Arduino_Pro_Mini:Arduino_Pro_Mini X1
+L TrialBBConversion-rescue:Arduino_Pro_Mini-Arduino_Pro_Mini X1
 U 1 1 5EE644F2
 P 6000 3600
